File: hardware/2port/thor-2port.kicad_pcb (KiCad board)
At the start: 2 copper layers, 93 x 65 mm, 19 parts, among them J1 THOR J47 / Wieson, J10 AUX / RAW IO, J11 RESERVED CAN / RAW, J12 SHIELD / GND / OPEN, J2 FSI_CAN0 / CAN, J3 FSI_CAN1 / CAN

Commit message: Revise A1 CAN routing, enclosure identity and engineering documentation
Parts:
- moved JP1 8.00 mm to (25.6, 19.0)
- moved JP2 8.00 mm to (67.6, 19.0)
- moved D1 5.42 mm to (27.6, 12.5), turned to 90 degrees
- moved D2 5.42 mm to (69.6, 12.5), turned to 90 degrees
Routing:
- net /GND: track 139.5 -> 71.7 mm, vias 2 -> 8
- net /AURIX_PWM_GPIO: track 42.0 -> 60.0 mm, vias 0 -> 1
- net /FSI_EXT_GPIO1: track 50.2 -> 67.9 mm, vias 0 -> 1
- net /FSI_CAN0_L: track 67.2 -> 52.9 mm, vias 1 -> 2
- net /AURIX_CAN2_TERM: track 34.6 -> 47.3 mm
- net /AURIX_SCL_TXD: track 48.4 -> 37.7 mm
- net /AURIX_CAN1_L: track 32.8 -> 42.0 mm, vias 0 -> 1
- net /FSI_CAN0_TERM: track 22.5 -> 30.5 mm, vias 0 -> 1
- net /FSI_CAN1_TERM: track 47.5 -> 55.4 mm
- net /FSI_CAN0_H: track 65.3 -> 57.4 mm, vias 1 -> 2
- net /HOST_5V_AO: track 38.7 -> 46.3 mm, vias 3 -> 1
- net /FSI_CAN1_L: track 86.4 -> 79.1 mm, vias 1 -> 2
- net /AURIX_CAN1_TERM: track 34.4 -> 41.3 mm
- net /AURIX_CAN2_H: track 38.7 -> 34.6 mm
- net /AURIX_CAN2_L: track 31.5 -> 34.1 mm, vias 0 -> 1
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- added copper zone on F.Cu, net /GND
Other:
- board text added: "THOR CAN 2 / A1 REVIEW"
- board text removed: "THOR CAN 2 / A0 REVIEW"

Commit message: Add prototype access, clear controls and reinforced mounting housings
Parts:
- added P1: ISOLATED PROTOTYPING PADS, Thor:Prototype_6x6_P2.54, F.Cu at (10.0, 72.0)
- added P2: ISOLATED PROTOTYPING PADS, Thor:Prototype_14x6_P2.54, F.Cu at (48.5, 72.0)
- added TP1: PROTO POWER / JP5-JP6 GATED, Thor:Prototype_Power_3x3_P2.54, F.Cu at (10.0, 62.0)
- added TP2: PROTO POWER / JP5-JP6 GATED, Thor:Prototype_Power_3x3_P2.54, F.Cu at (48.5, 62.0)
- moved H3 25.0 mm to (4.00, 86.0)
- moved H4 25.0 mm to (89.0, 86.0)
Routing:
- net /GND: track 71.7 -> 135.8 mm
- net /AUX_5V_AO: track 26.1 -> 85.6 mm, vias 0 -> 1
- net /AUX_3V3: track 29.5 -> 87.1 mm, vias 0 -> 1
Other:
- board size 93 x 65 mm -> 93 x 90 mm
- board text added: "10"
- board text added: "11"
- board text added: "12"
- board text added: "13"
- board text added: "14"
- board text added: "2"
- board text added: "3"
- board text added: "3V3"
- board text added: "4"
- board text added: "5"
- board text added: "5V"
- board text added: "6"
- board text added: "7"
- board text added: "8"
- board text added: "9"
- board text added: "A"
- board text added: "A1 DEV"
- board text added: "AUX: SHUNT = ON"
- board text added: "B"
- board text added: "C"
- board text added: "CAN0"
- board text added: "CAN0 TERM"
- board text added: "CAN1"
- board text added: "CAN1 TERM"
- board text added: "D"
- board text added: "DEFAULT OPEN"
- board text added: "E"
- board text added: "F"
- board text added: "FSI6"
- board text added: "FSI6: FSI FIRMWARE / NOT LINUX GPIO"
- board text added: "GND"
- board text added: "J10 RAW I/O"
- board text added: "J11 RESERVED"
- board text added: "JP1 = 120R"
- board text added: "JP2 = 120R"
- board text added: "KEEP CLEAR"
- board text added: "OPEN"
- board text added: "OUT1"
- board text added: "P1 / ISOLATED 2.54"
- board text added: "P2 / ISOLATED 2.54"
- board text added: "PGOOD"
- board text added: "PIN 9 NC / CAN ONLY"
- board text added: "PWM"
- board text added: "RIBBON"
- board text added: "SCL"
- board text added: "SDA"
- board text added: "SHIELD"
- board text added: "STOP1"
- board text added: "STOP2"
- board text added: "THOR CAN"
- board text added: "WAKE"
- board text added: "github.com/mvalancy"
- board text removed: "AUX RAW"
- board text removed: "FSI_CAN0"
- board text removed: "FSI_CAN1"
- board text removed: "PIN 9: NC / NOT RS232"
- board text removed: "TERM"
- board text removed: "THOR CAN 2 / A1 REVIEW"
